File: pcb/numitron_clock/numitron_clock.sch (KiCad schematic (older format))
At the start: 21 parts, among them J0 IV-9, J1 IV-9, J2 IV-9, J3 IV-9, J4 IV-9, J5 IV-9, J6 RTC, J7 PWR_JACK, U0 TPIC6595, U1 TPIC6595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

Commit message: not getting anywhere yet
Parts:
- removed C4, C5: 0.1uF, Capacitor_SMD:C_0805_2012Metric_Pad1.15x1.40mm_HandSolder, symbol Device:C
- removed J4, J5: IV-9, numitron_clock:NUM_IV-9, symbol Connector:Conn_01x09_Female
- removed U4, U5: TPIC6595, Package_SO:SOIC-20W_7.5x12.8mm_P1.27mm, symbol Interface_Expansion:TPIC6595
- A0: footprint (none) -> Module:Arduino_Nano
- J0, J1, J2, J3: footprint numitron_clock:NUM_IV-9 -> iv-9:NUM_IV-9
- J6: footprint (none) -> Connector_PinSocket_2.54mm:PinSocket_1x06_P2.54mm_Vertical; symbol Connector:Conn_01x04_Female -> Connector:Conn_01x06_Female
- J7: footprint (none) -> Connector_BarrelJack:BarrelJack_Horizontal
Connections:
- wire segments 171 -> 124
- no-connect marks 21 -> 23
